File: hardware/analogue_board/power.kicad_sch (KiCad schematic)
At the start: 47 parts, among them J201 Eurorack power 2x5 shrouded, U201 TPS54308DDCR, U202 L78M05ABDT-TR, U203 XC6206P332MR-G, U204 XC6206P332MR-G

Commit message: Analogue board: block review applied, TRS MIDI, ESP32-P4 support
Checkpoint 1 schematic rebuilt after a block-by-block prior-art review
(docs/analogue_board_review/, seven reports and an index).

Schematic:
- Codec: 20 Vpp in and out (15k input feedback; balanced MFB output,
  gain 2.5, 1 nF C0G); ferrite and 5.1 ohm on the codec supplies; VCOM
  decoupled at each input; CODEC_RST to a hole.
- Power: 680 ohm minimum load on +3V3D; buck input ferrite and EN
  divider; SS34 at D201-D203; Q201/JP201 MOD_5V bypass for the ESP32-P4.
- CV in: 15 V TVS at each jack, 1 nF at each ADC input, 1206 outputs.
- CV out: 12k/22k offset with 1 nF, 33k gain; CV7-8 feedback from the
  jack side of the 1k.
- Gates and panel: CS_595 pull-up, GATE_OE_N on J603, 1M wiper
  pull-downs, POT_REF, button RC order, 47 uF at the LED holes.
- New sheet 10: TRS MIDI (Type A), H11L1 in, 5 V buffered out.
- Layout: no overlapping text on any sheet.

ERC 0/0; netlist identical to intent (345 nets); 21 ICs against
datasheets; 17 Extended part types.

Spec v0.4: David's decisions (TVS yes, CV +/-5 V with a +/-10 V
variant, ESP32-P4 accommodated, power header free to move), the
corrections, and a firmware requirements list in section 15.

Co-Authored-By: Claude Opus 5.5 <noreply@anthropic.com>
Parts:
- removed D203: SS14, Diode_SMD:D_SMA, symbol Diode:SS14
- removed R203: 0R, Resistor_SMD:R_0805_2012Metric, symbol Device:R_Small
- added C211: 22u 25V, Capacitor_SMD:C_1206_3216Metric, symbol Device:C_Small
- added C222: 10u 25V, Capacitor_SMD:C_0805_2012Metric, symbol Device:C_Small
- added D203: SS34, Diode_SMD:D_SMA, symbol Diode:SS34
- added FB203: BLM18PG121, Inductor_SMD:L_0603_1608Metric, symbol Device:FerriteBead_Small
- added JP201: ESP32-P4: bridge, Jumper:SolderJumper-2_P1.3mm_Open_RoundedPad1.0x1.5mm, symbol Jumper:SolderJumper_2_Open
- added Q201: AO3401A, Package_TO_SOT_SMD:SOT-23, symbol Transistor_FET:AO3401A
- added R207, R208, R209: 0R, Resistor_SMD:R_0603_1608Metric, symbol Device:R_Small
- added R210: 680R, Resistor_SMD:R_0603_1608Metric, symbol Device:R_Small
- added R211: 1M, Resistor_SMD:R_0402_1005Metric, symbol Device:R_Small
- added R212: 100k, Resistor_SMD:R_0402_1005Metric, symbol Device:R_Small
- C206: value 100n 50V -> 10u 50V; footprint Capacitor_SMD:C_0603_1608Metric -> Capacitor_SMD:C_1206_3216Metric; Dielectric X7R -> X5R; LCSC C14663 -> C13585
- C207: value 100n 16V -> 100n 50V; footprint Capacitor_SMD:C_0402_1005Metric -> Capacitor_SMD:C_0603_1608Metric; Decouples (none) -> U201 VIN pin 3; LCSC C1525 -> C14663; Note bootstrap -> (none); Voltage 16V -> 50V
- C208: value 47p 50V -> 100n 16V; Dielectric C0G -> X7R; LCSC C1567 -> C1525; Note feed-forward, fit only if the loop needs phase boost -> bootstrap; Voltage 50V -> 16V; now fitted
- C209: value 22u 25V -> 470p 50V; footprint Capacitor_SMD:C_1206_3216Metric -> Capacitor_SMD:C_0402_1005Metric; Decouples buck output -> (none); Dielectric X5R -> C0G; JLC Basic -> not fitted; LCSC C12891 -> (none); Note (none) -> feed-forward, fit only if the loop needs phase boost (TI ta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; Voltage 25V -> 50V; now not fitted
- C212: value 10u 25V -> 100n 16V; footprint Capacitor_SMD:C_0805_2012Metric -> Capacitor_SMD:C_0402_1005Metric; Decouples +5VD distribution -> buck output; Dielectric X5R -> X7R; LCSC C15850 -> C1525; Voltage 25V -> 16V
- C213: value 1u 50V -> 10u 25V; footprint Capacitor_SMD:C_0603_1608Metric -> Capacitor_SMD:C_0805_2012Metric; Decouples U202 VI pin 1 -> +5VD distribution; LCSC C15849 -> C15850; Voltage 50V -> 25V
- C214: value 100n 50V -> 1u 50V; Dielectric X7R -> X5R; LCSC C14663 -> C15849
- C215: value 10u 25V -> 100n 50V; footprint Capacitor_SMD:C_0805_2012Metric -> Capacitor_SMD:C_0603_1608Metric; Decouples U202 output -> U202 VI pin 1; Dielectric X5R -> X7R; LCSC C15850 -> C14663; Voltage 25V -> 50V
- C216: value 100n 16V -> 10u 25V; footprint Capacitor_SMD:C_0402_1005Metric -> Capacitor_SMD:C_0805_2012Metric; Dielectric X7R -> X5R; LCSC C1525 -> C15850; Voltage 16V -> 25V
- C217: value 1u 25V -> 100n 16V; Decouples U203 VI pin 3 -> U202 output; Dielectric X5R -> X7R; LCSC C52923 -> C1525; Voltage 25V -> 16V
- C218: value 10u 25V -> 1u 25V; footprint Capacitor_SMD:C_0805_2012Metric -> Capacitor_SMD:C_0402_1005Metric; Decouples U203 output (ceramic-stable LDO) -> U203 VI pin 3; LCSC C15850 -> C52923
- C219: value 1u 25V -> 10u 25V; footprint Capacitor_SMD:C_0402_1005Metric -> Capacitor_SMD:C_0805_2012Metric; Decouples U204 VI pin 3 -> U203 output (ceramic-stable LDO); LCSC C52923 -> C15850
- C220: value 10u 25V -> 1u 25V; footprint Capacitor_SMD:C_0805_2012Metric -> Capacitor_SMD:C_0402_1005Metric; Decouples U204 output (ceramic-stable LDO) -> U204 VI pin 3; LCSC C15850 -> C52923
- C221: Decouples module supply: A101 VSYS pin 39, A102 VIN pin 48 -> U204 output (ceramic-stable LDO)
- D201, D202: value SS14 -> SS34; symbol Diode:SS14 -> Diode:SS34; LCSC C2480 -> C8678; MPN SS14 -> SS34
- R201: value 15k -> 510k; footprint Resistor_SMD:R_0402_1005Metric -> Resistor_SMD:R_0603_1608Metric; LCSC C25756 -> C23192; Note (none) -> EN divider (UVLO), top
- R202: value 2k -> 75k; footprint Resistor_SMD:R_0402_1005Metric -> Resistor_SMD:R_0603_1608Metric; LCSC C4109 -> C23242; Note (none) -> EN divider (UVLO), bottom
- R203: renamed from C211; value 100n 16V -> 15k; footprint Capacitor_SMD:C_0402_1005Metric -> Resistor_SMD:R_0402_1005Metric; symbol Device:C_Small -> Device:R_Small; Decouples buck output -> (none); Dielectric X7R -> (none); LCSC C1525 -> C25756; Tolerance (none) -> 1%; Voltage 16V -> (none)
- R204: value 0R -> 2k; footprint Resistor_SMD:R_0603_1608Metric -> Resistor_SMD:R_0402_1005Metric; LCSC C21189 -> C4109; Note rail link: lift to isolate +5VA -> (none)
- R205: value 0R -> 2k; footprint Resistor_SMD:R_0603_1608Metric -> Resistor_SMD:R_0402_1005Metric; LCSC C21189 -> C4109; Note rail link: lift to isolate +3V3A -> feed-forward series resistor, fit with the capacitor; now not fitted
- R206: footprint Resistor_SMD:R_0603_1608Metric -> Resistor_SMD:R_0805_2012Metric; LCSC C21189 -> C17477; Note rail link: lift to isolate +3V3D -> rail link: lift to isolate +5VD
Connections:
- net +12V: now also C215.1, FB203.1; no longer C205.1, C206.1, C213.1, U201.3 (VIN)
- net +3V3A: now also R208.2; no longer R205.2
- net +3V3D: now also R209.2, R210.1; no longer R206.2
- net +5VA: now also C218.1, R207.2; no longer C217.1, R204.2
- net +5VD: now also C213.1, C220.1, R206.2, D203.2 (A), Q201.3 (D); no longer C212.1, C219.1
- net 3V3A_REG: now also C219.1, R208.1; no longer C218.1, R205.1
- net 3V3D_REG: now also C221.1, R209.1; no longer C220.1, R206.1
- net 5VA_REG: now also C217.1, R207.1; no longer C215.1, R204.1
- net 5V_BUCK: now also C212.1, R206.1, C211.1; no longer C208.1, R201.1
- net GND: now also C207.2, R204.2, C211.2, C222.2, R210.2, R212.2; no longer C209.2, R203.2
- net MOD_5V: now also C222.1, D203.1 (K), Q201.2 (S), R211.1; no longer C221.1
- net at L201.1, U201.2 (SW): now also C208.2; no longer C207.2
- net BUCK_EN: now reaches R201.2, R202.1
- net BUCK_EN: now also U201.5 (EN); no longer C208.2, U201.4 (FB)
- net at U201.6 (BOOT): now also C208.1; no longer C207.1
- new net: R203.2, R204.1, R205.2, U201.4 (FB)
- new net: C209.2, R205.1
- new net BUCK_VIN: C205.1, C206.1, C207.1, FB203.2, R201.1, U201.3 (VIN)
- new net FET_EN: JP201.2 (B), R212.1
- new net PICO_VBUS: JP201.1 (A), Q201.1 (G), R211.2
- no-connect marks 1 -> 0
Other:
- note added: "+3V3A: XC6206 from +5VA (DAC8568, MCP3208, pot reference via POT_REF)"
- note added: "+3V3D: XC6206 from +5VD (codec VDD, ADS8688 DVDD, logic, Qwiic, MIDI)"
- note added: "680 Ω minimum load: four 12 V gates push ≈3.4 mA into +3V3D through their clamps; the XC6206 cannot sink it (4.85 mA here)."
- note added: "Load estimate: +12 V ≈ 120 mA typical, ~350 mA worst case with a Teensy and a lit LED chain; with an ESP32-P4 (0.45-0.7 A at 5 V) plus LEDs, ≈0.75 A. -12 V ≈ 25 mA. XC6206: 200 mA each; +3V3D ≈ 50 mA."
- note added: "MOD_5V: +5VD through a Schottky to Pico VSYS / Teensy VIN / ESP32-P4 VCC_5V"
- note added: "Q201 bypasses D203 when JP201 is bridged, for the ESP32-P4, whose regulator needs ≥ 4.5 V at 0.5-0.7 A. Its gate follows the Pico/P4 VBUS pin (pin 40): with USB plugged in the FET turns off, as in the Pico 2 datasheet's VSYS circuit. Leave JP201 open for a Teensy (an uncut VIN-VUSB link would tie USB to the buck)."
- note added: "SS34 per rail: reverse-polarity protection. A reversed ribbon blocks on both rails. 3 A parts: +12 V can reach ≈0.75 A with an ESP32-P4 and a lit LED chain."
- note added: "Vout = 0.596 V × (1 + 15k/2k) = 5.07 V; L and Cout from TI's table for 5 V. Input: own ferrite and 2 × 10 µF, keeping the 350 kHz input ripple off the ±12 V rail the op-amps share. EN divider 510k/75k: starts at ≈9.2 V, stops at ≈8.1 V, so the digital 5 V never runs while the analogue 5 V (L78M05) is down: TI's power-up order for the codec."
- note removed: "+3V3A: XC6206 from +5VA (DAC8568, MCP3208 and pot reference)"
- note removed: "+3V3D: XC6206 from +5VD (codec VDD, ADS8688 DVDD, logic, Qwiic)"
- note removed: "Load estimate: +12 V ≈ 120 mA typical, ~350 mA worst case (Teensy at full clock plus a lit LED chain through the buck); -12 V ≈ 25 mA (op-amps). XC6206: 200 mA each; +3V3D ≈ 50 mA, +3V3A ≈ 6 mA."
- note removed: "MOD_5V: +5VD through a Schottky to Pico VSYS / Teensy VIN"
- note removed: "SS14 per rail: reverse-polarity protection. A reversed ribbon blocks on both rails."
- note removed: "Vout = 0.596 V × (1 + 15k/2k) = 5.07 V. L and Cout from TI's table for 5 V. EN floats (internal pull-up) = on."
- moved on the sheet: U201
