File: hardware/analogue_board/analogue_board.kicad_sch (KiCad schematic)
At the start: 3 parts, among them J101 Spare GPIO, Pico RUN

Commit message: Analogue board: block review applied, TRS MIDI, ESP32-P4 support
Checkpoint 1 schematic rebuilt after a block-by-block prior-art review
(docs/analogue_board_review/, seven reports and an index).

Schematic:
- Codec: 20 Vpp in and out (15k input feedback; balanced MFB output,
  gain 2.5, 1 nF C0G); ferrite and 5.1 ohm on the codec supplies; VCOM
  decoupled at each input; CODEC_RST to a hole.
- Power: 680 ohm minimum load on +3V3D; buck input ferrite and EN
  divider; SS34 at D201-D203; Q201/JP201 MOD_5V bypass for the ESP32-P4.
- CV in: 15 V TVS at each jack, 1 nF at each ADC input, 1206 outputs.
- CV out: 12k/22k offset with 1 nF, 33k gain; CV7-8 feedback from the
  jack side of the 1k.
- Gates and panel: CS_595 pull-up, GATE_OE_N on J603, 1M wiper
  pull-downs, POT_REF, button RC order, 47 uF at the LED holes.
- New sheet 10: TRS MIDI (Type A), H11L1 in, 5 V buffered out.
- Layout: no overlapping text on any sheet.

ERC 0/0; netlist identical to intent (345 nets); 21 ICs against
datasheets; 17 Extended part types.

Spec v0.4: David's decisions (TVS yes, CV +/-5 V with a +/-10 V
variant, ESP32-P4 accommodated, power header free to move), the
corrections, and a firmware requirements list in section 15.

Co-Authored-By: Claude Opus 5.5 <noreply@anthropic.com>
Parts:
- J101: value Spare GPIO, Pico RUN -> Spare GPIO, MIDI links, Pico RUN; footprint Connector_PinHeader_2.54mm:PinHeader_1x04_P2.54mm_Vertical -> Connector_PinHeader_2.54mm:PinHeader_1x06_P2.54mm_Vertical; symbol Connector_Generic:Conn_01x04 -> Connector_Generic:Conn_01x06
Connections:
- net GND: now also J101.6 (Pin_6); no longer J101.4 (Pin_4)
- net RUN: now also J101.5 (Pin_5); no longer J101.3 (Pin_3)
- net SPARE2: now also J101.3 (Pin_3); no longer J101.2 (Pin_2)
- net PICO_VBUS: now reaches A101.40 (VBUS)
- new net MIDI_RX: J101.4 (Pin_4)
- new net MIDI_TX: J101.2 (Pin_2)
- no-connect marks 22 -> 21
Other:
- added sheet TRS MIDI (midi.kicad_sch)
- note added: "Both footprints sit on the one board, wired to the same nets; only one module is fitted. Every signal into a module is 3.3 V: the Teensy 4.1 is not 5 V tolerant. Pico 2: 5 V reaches VSYS through D203 (Schottky, net MOD_5V), VBUS is left to USB. Teensy 4.1: cut the VIN–VUSB pads before fitting; VIN takes MOD_5V. Neither module's own 3.3 V output is used: the board makes its own +3V3A and +3V3D. ES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"
- note added: "MIDI in (H11L1) and out (5 V buffered), Type A"
- note added: "MIDI: bridge SPARE1-MIDI_TX and SPARE2-MIDI_RX (adjacent holes) with a wire or shunt. Left open, SPARE1/2 are plain GPIO. On a Pico, move the SDK console off UART0 to USB. RUN: wire a reset button to GND (Pico or ESP32-P4)."
- note removed: "Both footprints sit on the one board, wired to the same nets; only one module is fitted. Every signal into a module is 3.3 V: the Teensy 4.1 is not 5 V tolerant. Pico 2: 5 V reaches VSYS through D203 (Schottky, net MOD_5V), VBUS is left to USB. Teensy 4.1: cut the VIN–VUSB pads before fitting; VIN takes MOD_5V. Neither module's own 3.3 V output is used: the board makes its own +3V3A and +3V3D."
- note removed: "RUN: wire a reset button to GND (Pico only; the Teensy has no reset at its edge)."

Commit message: Analogue board: checkpoint 3 started; double-sided, floorplan placed
- pcb.py generates analogue_board.kicad_pcb from the netlist: outline,
  JLC 4-layer stack-up, every footprint with nets and schematic links
  (KiCad schematic parity: 0 differences), parked parts beside the board,
  courtyard area budget, DRC and 3D renders of both faces.
- Area budget: the courtyards need 104% of one face before routing, so
  David chose double-sided assembly (JLC Standard PCBA, about $100 more
  per order, to confirm on a quote).
- Floorplan in placement.py: analogue ICs at the top under the modules,
  furthest from the buck; logic below; power bottom right around J201;
  MIDI bottom left; 99 wiring-field holes in three columns lined up with
  the edge-strip positions, each group beside its circuit.
- Library: module socket courtyards cover only their header rows; the
  wiring holes get their own footprint with a one-pitch courtyard.
- Spec records the decision, the floorplan and David's answers: 11 mm to
  the deck in 10HP (deck parts 2 mm at most); holes tinned both faces.

Co-Authored-By: Claude Opus 5.5 <noreply@anthropic.com>
Parts:
- J101: footprint Connector_PinHeader_2.54mm:PinHeader_1x06_P2.54mm_Vertical -> analogue_board:WiringHoles_1x06
Changed lines of the file:
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@@
 			)
 		)
-		(property "Footprint" "Connector_PinHeader_2.54mm:PinHeader_1x06_P2.54mm_Vertical"
+		(property "Footprint" "analogue_board:WiringHoles_1x06"
 			(at 74.93 170.18 0)
 			(effects
