File: hardware/analogue_board/cv_dac.kicad_sch (KiCad schematic)
At the start: 41 parts, among them U501 DAC8568IAPWR, U502 TL074HIDR, U503 TL074HIDR, U504 TL074HIDR

Commit message: Analogue board: block review applied, TRS MIDI, ESP32-P4 support
Checkpoint 1 schematic rebuilt after a block-by-block prior-art review
(docs/analogue_board_review/, seven reports and an index).

Schematic:
- Codec: 20 Vpp in and out (15k input feedback; balanced MFB output,
  gain 2.5, 1 nF C0G); ferrite and 5.1 ohm on the codec supplies; VCOM
  decoupled at each input; CODEC_RST to a hole.
- Power: 680 ohm minimum load on +3V3D; buck input ferrite and EN
  divider; SS34 at D201-D203; Q201/JP201 MOD_5V bypass for the ESP32-P4.
- CV in: 15 V TVS at each jack, 1 nF at each ADC input, 1206 outputs.
- CV out: 12k/22k offset with 1 nF, 33k gain; CV7-8 feedback from the
  jack side of the 1k.
- Gates and panel: CS_595 pull-up, GATE_OE_N on J603, 1M wiper
  pull-downs, POT_REF, button RC order, 47 uF at the LED holes.
- New sheet 10: TRS MIDI (Type A), H11L1 in, 5 V buffered out.
- Layout: no overlapping text on any sheet.

ERC 0/0; netlist identical to intent (345 nets); 21 ICs against
datasheets; 17 Extended part types.

Spec v0.4: David's decisions (TVS yes, CV +/-5 V with a +/-10 V
variant, ESP32-P4 accommodated, power header free to move), the
corrections, and a firmware requirements list in section 15.

Co-Authored-By: Claude Opus 5.5 <noreply@anthropic.com>
Parts:
- removed C512: 100p 50V, Capacitor_SMD:C_0402_1005Metric, symbol Device:C_Small
- removed unit 4 of U503
- removed unit 4 of U504
- added C518: 100n 50V, Capacitor_SMD:C_0603_1608Metric, symbol Device:C_Small
- added R518, R521: 33k, Resistor_SMD:R_0402_1005Metric, symbol Device:R_Small
- added R520: 1k, Resistor_SMD:R_1206_3216Metric, symbol Device:R_Small
- added unit 2 of U504
- C504: value 1u 25V -> 1n 50V; Dielectric X5R -> X7R; LCSC C52923 -> C1523; Note 24 Hz filter on the offset reference -> light filter; must follow VREF at enable; Voltage 25V -> 50V
- C512: renamed from U504; value TL074HIDR -> 100p 50V; footprint Package_SO:SOIC-14_3.9x8.7mm_P1.27mm -> Capacitor_SMD:C_0402_1005Metric; symbol Amplifier_Operational:TL074 -> Device:C_Small; Dielectric (none) -> C0G; JLC Extended -> Basic; LCSC C2878713 -> C1546; MPN TL074HIDR -> (none); Voltage (none) -> 50V
- C513: renamed from C514; Decouples U502 V- pin 11 -> U502 V+ pin 4
- C514: renamed from U503; value TL074HIDR -> 100n 50V; footprint Package_SO:SOIC-14_3.9x8.7mm_P1.27mm -> Capacitor_SMD:C_0603_1608Metric; symbol Amplifier_Operational:TL074 -> Device:C_Small; Decouples (none) -> U502 V- pin 11; Dielectric (none) -> X7R; JLC Extended -> Basic; LCSC C2878713 -> C14663; MPN TL074HIDR -> (none); Voltage (none) -> 50V
- C515: renamed from C516; Decouples U503 V- pin 11 -> U503 V+ pin 4
- C516: renamed from U504; value TL074HIDR -> 100n 50V; footprint Package_SO:SOIC-14_3.9x8.7mm_P1.27mm -> Capacitor_SMD:C_0603_1608Metric; symbol Amplifier_Operational:TL074 -> Device:C_Small; Decouples (none) -> U503 V- pin 11; Dielectric (none) -> X7R; JLC Extended -> Basic; LCSC C2878713 -> C14663; MPN TL074HIDR -> (none); Voltage (none) -> 50V
- C517: renamed from C518; Decouples U504 V- pin 11 -> U504 V+ pin 4
- R502: value 10k -> 12k; LCSC C25744 -> C25752
- R503: value 20k -> 22k; LCSC C25765 -> C25768
- R504, R506, R508, R510, R512, R514, R516: value 30k -> 10k; footprint Resistor_SMD:R_0603_1608Metric -> Resistor_SMD:R_0402_1005Metric; LCSC C22984 -> C25744
- R505, R507, R509, R511, R513, R515: value 10k -> 33k; LCSC C25744 -> C25779
- R517: value 10k -> 1k; footprint Resistor_SMD:R_0402_1005Metric -> Resistor_SMD:R_1206_3216Metric; LCSC C25744 -> C4410; Note (none) -> inside the feedback loop; 1206 for patching faults
- U502: renamed from C513; value 100n 50V -> TL074HIDR; footprint Capacitor_SMD:C_0603_1608Metric -> Package_SO:SOIC-14_3.9x8.7mm_P1.27mm; symbol Device:C_Small -> Amplifier_Operational:TL074; Decouples U502 V+ pin 4 -> (none); Dielectric X7R -> (none); JLC Basic -> Extended; LCSC C14663 -> C2878713; MPN (none) -> TL074HIDR; Voltage 50V -> (none)
- U503: renamed from C515; value 100n 50V -> TL074HIDR; footprint Capacitor_SMD:C_0603_1608Metric -> Package_SO:SOIC-14_3.9x8.7mm_P1.27mm; symbol Device:C_Small -> Amplifier_Operational:TL074; Decouples U503 V+ pin 4 -> (none); Dielectric X7R -> (none); JLC Basic -> Extended; LCSC C14663 -> C2878713; MPN (none) -> TL074HIDR; Voltage 50V -> (none)
- U503: renamed from R518; value 30k -> TL074HIDR; footprint Resistor_SMD:R_0603_1608Metric -> Package_SO:SOIC-14_3.9x8.7mm_P1.27mm; symbol Device:R_Small -> Amplifier_Operational:TL074; JLC Basic -> Extended; LCSC C22984 -> C2878713; MPN (none) -> TL074HIDR; Tolerance 1% -> (none)
- U504: renamed from C517; value 100n 50V -> TL074HIDR; footprint Capacitor_SMD:C_0603_1608Metric -> Package_SO:SOIC-14_3.9x8.7mm_P1.27mm; symbol Device:C_Small -> Amplifier_Operational:TL074; Decouples U504 V+ pin 4 -> (none); Dielectric X7R -> (none); JLC Basic -> Extended; LCSC C14663 -> C2878713; MPN (none) -> TL074HIDR; Voltage 50V -> (none)
- renumbered U502 to U504
Connections:
- net +12V: now also C513.1, C515.1, C517.1, U502.4 (V+), U503.4 (V+), U504.4 (V+); no longer C514.4 (V+), C516.4 (V+), U502.1, U503.1, U504.1, U504.4 (V+)
- net -12V: now also C514.1, C516.1, U502.11 (V-), U503.11 (V-), U504.11 (V-), C518.1; no longer C513.1, C514.11 (V-), C515.1, C516.11 (V-), C517.1, U504.11 (V-)
- net CVDRV1: now also R505.2; no longer R504.2
- net CVDRV2: now also R507.2; no longer R506.2
- net CVDRV3: now also R509.2; no longer R508.2
- net CVDRV4: now also R511.2; no longer R510.2
- net CVDRV5: now also R513.2; no longer R512.2
- net CVDRV6: now also R515.2; no longer R514.2
- net DAC8: now also U503.12 (+)
- net GND: now also C514.2, C516.2, U504.12 (+), C518.2, U504.5 (+); no longer C512.5 (+), U502.2, U503.2, U504.2
- net OFFSET_REF: now also R504.1, R506.1, R508.1, R510.1, R512.1, R514.1, R516.1; no longer R505.1, R507.1, R509.1, R511.1, R513.1, R515.1, R517.1
- net at C509.1, U503.2 (-): now also R512.2, R513.1; no longer R512.1, R513.2
- net at C506.1, U502.6 (-): now also R506.2, R507.1; no longer R506.1, R507.2
- net at C508.1, U502.13 (-): now also R510.2, R511.1; no longer R510.1, R511.2
- net at C507.1, U502.9 (-): now also R508.2, R509.1; no longer R508.1, R509.2
- net at C510.1, U503.6 (-): now also R514.2, R515.1; no longer R514.1, R515.2
- net at C505.1, U502.2 (-): now also R504.2, R505.1; no longer R504.1, R505.2
- net at C511.1, U503.9 (-): now also R516.2, R518.1; no longer R516.1, R517.2
- net at R519.2: now also C512.1, U503.13 (-), R521.1; no longer U503.1
- net CVDRV7: no longer names the net of C511.2, U503.8
- net CVDRV7: now also R517.1; no longer R516.2
- removed net CVDRV8: U503.2
- new net: C512.2, R520.1, U503.14
- new net: U504.6 (-), U504.7
- new net: U504.13 (-), U504.14
- new net CVO7: R517.2, R518.2
- new net CVO8: R520.2, R521.2
Other:
- note added: "1 nF (not 1 µF): the offset must track VREF quickly, or enabling the reference glitches every output."
- note added: "CVDRV1-6 go to the DG412 switches (sheet CV jacks & ADC). CVO7-8 go straight to their holes."
- note added: "DAC8568 grade A: 0-2.5 V from its internal reference (off at power-up), outputs reset to zero. Each stage: non-inverting gain 1 + 33k/10k = 4.3, offset by OFFSET_REF = VREF × 22k/34k through the 10 kΩ: Vout = 4.3·Vdac − 5.34 V, so −5.34 V … +5.41 V, putting ±5 V inside the DAC's specified codes (0 V at code ≈ 32544). The offset tracks the DAC's own reference, as in Performer, O&C, Marbles and Sta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"
- note added: "OFFSET_REF = VREF × 22k/(12k + 22k) = 1.618 V, buffered"
- note removed: "CVDRV1-6 go to the DG412 switches; CVDRV7-8 straight to their jacks through 1 kΩ (sheet CV jacks & ADC)."
- note removed: "DAC8568 grade A: 0-2.5 V from its internal reference (off at power-up; firmware enables it), outputs reset to zero. Each stage: non-inverting gain 1 + 30k/10k = 4, offset by OFFSET_REF = 2/3 × VREF through the 10 kΩ: Vout = 4·Vdac − 3·(2/3)·VREF = −5 V … +5 V. The offset tracks the DAC's own reference, so mid-code is 0 V whatever the reference does. Before the reference is on, OFFSET_REF is 0 V a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"
- note removed: "OFFSET_REF = VREF × 20k/(10k + 20k) = 1.667 V, buffered"
- moved on the sheet: C513, C515, C517
