File: hardware/analogue_board/midi.kicad_sch (KiCad schematic)
At the start: 17 parts, among them J1001 TRS MIDI holes, U1001 SN74AHCT1G125DBVR, U1002 H11L1SR2M

Commit message: Analogue board: checkpoint 3 started; double-sided, floorplan placed
- pcb.py generates analogue_board.kicad_pcb from the netlist: outline,
  JLC 4-layer stack-up, every footprint with nets and schematic links
  (KiCad schematic parity: 0 differences), parked parts beside the board,
  courtyard area budget, DRC and 3D renders of both faces.
- Area budget: the courtyards need 104% of one face before routing, so
  David chose double-sided assembly (JLC Standard PCBA, about $100 more
  per order, to confirm on a quote).
- Floorplan in placement.py: analogue ICs at the top under the modules,
  furthest from the buck; logic below; power bottom right around J201;
  MIDI bottom left; 99 wiring-field holes in three columns lined up with
  the edge-strip positions, each group beside its circuit.
- Library: module socket courtyards cover only their header rows; the
  wiring holes get their own footprint with a one-pitch courtyard.
- Spec records the decision, the floorplan and David's answers: 11 mm to
  the deck in 10HP (deck parts 2 mm at most); holes tinned both faces.

Co-Authored-By: Claude Opus 5.5 <noreply@anthropic.com>
Parts:
- J1001: footprint Connector_PinHeader_2.54mm:PinHeader_1x06_P2.54mm_Vertical -> analogue_board:WiringHoles_1x06
Changed lines of the file:
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@@
 			)
 		)
-		(property "Footprint" "Connector_PinHeader_2.54mm:PinHeader_1x06_P2.54mm_Vertical"
+		(property "Footprint" "analogue_board:WiringHoles_1x06"
 			(at 200.66 101.6 0)
 			(effects
