File: hardware/analogue_board/codec_audio.kicad_sch (KiCad schematic)
At the start: 50 parts, among them J301 Audio in holes, J302 Audio out holes, U301 PCM3060PWR, U302 TL074HIDR

Commit message: Analogue board: block review applied, TRS MIDI, ESP32-P4 support
Checkpoint 1 schematic rebuilt after a block-by-block prior-art review
(docs/analogue_board_review/, seven reports and an index).

Schematic:
- Codec: 20 Vpp in and out (15k input feedback; balanced MFB output,
  gain 2.5, 1 nF C0G); ferrite and 5.1 ohm on the codec supplies; VCOM
  decoupled at each input; CODEC_RST to a hole.
- Power: 680 ohm minimum load on +3V3D; buck input ferrite and EN
  divider; SS34 at D201-D203; Q201/JP201 MOD_5V bypass for the ESP32-P4.
- CV in: 15 V TVS at each jack, 1 nF at each ADC input, 1206 outputs.
- CV out: 12k/22k offset with 1 nF, 33k gain; CV7-8 feedback from the
  jack side of the 1k.
- Gates and panel: CS_595 pull-up, GATE_OE_N on J603, 1M wiper
  pull-downs, POT_REF, button RC order, 47 uF at the LED holes.
- New sheet 10: TRS MIDI (Type A), H11L1 in, 5 V buffered out.
- Layout: no overlapping text on any sheet.

ERC 0/0; netlist identical to intent (345 nets); 21 ICs against
datasheets; 17 Extended part types.

Spec v0.4: David's decisions (TVS yes, CV +/-5 V with a +/-10 V
variant, ESP32-P4 accommodated, power header free to move), the
corrections, and a firmware requirements list in section 15.

Co-Authored-By: Claude Opus 5.5 <noreply@anthropic.com>
Parts:
- removed C307, C312: 100p 50V, Capacitor_SMD:C_0402_1005Metric, symbol Device:C_Small
- removed D301: BAT54S, Package_TO_SOT_SMD:SOT-23, symbol Diode:BAT54S
- removed R314, R317: 15k, Resistor_SMD:R_0402_1005Metric, symbol Device:R_Small
- removed R318: 1k, Resistor_SMD:R_0402_1005Metric, symbol Device:R_Small
- removed unit 1 of U302
- added C310, C317: 100p 50V, Capacitor_SMD:C_0402_1005Metric, symbol Device:C_Small
- added C311: 1u 50V, Capacitor_SMD:C_0805_2012Metric, symbol Device:C_Small
- added C315, C318: 1n C0G 50V, Capacitor_SMD:C_0603_1608Metric, symbol Device:C_Small
- added C319, C320: 100n 50V, Capacitor_SMD:C_0603_1608Metric, symbol Device:C_Small
- added FB301: BLM18PG121, Inductor_SMD:L_0603_1608Metric, symbol Device:FerriteBead_Small
- added J303: Codec RST, Connector_PinHeader_2.54mm:PinHeader_1x02_P2.54mm_Vertical, symbol Connector_Generic:Conn_01x02
- added R308: 100k, Resistor_SMD:R_0402_1005Metric, symbol Device:R_Small
- added R309: 1M, Resistor_SMD:R_0402_1005Metric, symbol Device:R_Small
- added R316: 12k, Resistor_SMD:R_0402_1005Metric, symbol Device:R_Small
- added R321: 1k, Resistor_SMD:R_1206_3216Metric, symbol Device:R_Small
- added R324, R325: 1k, Resistor_SMD:R_0402_1005Metric, symbol Device:R_Small
- added R326, R327: 30k, Resistor_SMD:R_0603_1608Metric, symbol Device:R_Small
- added TP302: BCK, TestPoint:TestPoint_Pad_D1.0mm, symbol Connector:TestPoint
- C307: renamed from R309; value 1k -> 100p 50V; footprint Resistor_SMD:R_0402_1005Metric -> Capacitor_SMD:C_0402_1005Metric; symbol Device:R_Small -> Device:C_Small; Dielectric (none) -> C0G; LCSC C11702 -> C1546; Tolerance 1% -> (none); Voltage (none) -> 50V
- C309: value 100p 50V -> 100n 16V; Decouples (none) -> VCOM at U302 pin 3; Dielectric C0G -> X7R; LCSC C1546 -> C1525; Voltage 50V -> 16V
- C312: renamed from C311; value 100p 50V -> 100n 16V; Decouples (none) -> VCOM at U302 pin 5; Dielectric C0G -> X7R; LCSC C1546 -> C1525; Voltage 50V -> 16V
- C313: renamed from R322; value 15k -> 100p 50V; footprint Resistor_SMD:R_0402_1005Metric -> Capacitor_SMD:C_0402_1005Metric; symbol Device:R_Small -> Device:C_Small; Dielectric (none) -> C0G; LCSC C25756 -> C1546; Tolerance 1% -> (none); Voltage (none) -> 50V
- C316: value 100n 50V -> 100p 50V; footprint Capacitor_SMD:C_0603_1608Metric -> Capacitor_SMD:C_0402_1005Metric; Decouples U302 V- pin 11 -> (none); Dielectric X7R -> C0G; LCSC C14663 -> C1546
- D301: renamed from C310; value 1u 50V -> BAT54S; footprint Capacitor_SMD:C_0805_2012Metric -> Package_TO_SOT_SMD:SOT-23; symbol Device:C_Small -> Diode:BAT54S; Dielectric X7R -> (none); JLC Basic -> Extended; LCSC C28323 -> C408389; MPN (none) -> BAT54S; Note AC coupling, 50 V X7R -> (none); Voltage 50V -> (none)
- R304: value 1k -> 5.1R; footprint Resistor_SMD:R_0402_1005Metric -> Resistor_SMD:R_0603_1608Metric; LCSC C11702 -> C25197; Note RST pull-up (internal 50 kΩ pull-down) -> isolates the codec VDD from logic noise on +3V3D
- R305: value 220k -> 1k; footprint Resistor_SMD:R_0603_1608Metric -> Resistor_SMD:R_0402_1005Metric; LCSC C22961 -> C11702; Note MODE: 220 kΩ ±5 % to DGND selects H/W mode, differential out -> RST pull-up (internal 50 kΩ pull-down)
- R306: value 33k -> 220k; footprint Resistor_SMD:R_0402_1005Metric -> Resistor_SMD:R_0603_1608Metric; LCSC C25779 -> C22961; Note (none) -> MODE: 220 kΩ ±5 % to DGND selects H/W mode, differential out
- R307, R311: value 100k -> 15k; LCSC C25741 -> C25756
- R310: value 33k -> 1k; LCSC C25779 -> C11702
- R312: value 1M -> 100k; LCSC C26083 -> C25741; Note holds the jack side at 0 V -> (none)
- R313: value 1k -> 1M; LCSC C11702 -> C26083; Note (none) -> holds the jack side at 0 V
- R314: renamed from R316; value 12k -> 1k; LCSC C25752 -> C11702
- R317: renamed from R319; value 15k -> 1k; LCSC C25756 -> C11702
- R318: renamed from C313; value 100p 50V -> 1k; footprint Capacitor_SMD:C_0402_1005Metric -> Resistor_SMD:R_0402_1005Metric; symbol Device:C_Small -> Device:R_Small; Dielectric C0G -> (none); LCSC C1546 -> C11702; Tolerance (none) -> 1%; Voltage 50V -> (none)
- R319: renamed from R320; value 12k -> 30k; footprint Resistor_SMD:R_0402_1005Metric -> Resistor_SMD:R_0603_1608Metric; LCSC C25752 -> C22984
- R320: renamed from R321; value 12k -> 30k; footprint Resistor_SMD:R_0402_1005Metric -> Resistor_SMD:R_0603_1608Metric; LCSC C25752 -> C22984
- R322: renamed from C315; value 100n 50V -> 12k; footprint Capacitor_SMD:C_0603_1608Metric -> Resistor_SMD:R_0402_1005Metric; symbol Device:C_Small -> Device:R_Small; Decouples U302 V+ pin 4 -> (none); Dielectric X7R -> (none); LCSC C14663 -> C25752; Tolerance (none) -> 1%; Voltage 50V -> (none)
- R323: value 1k -> 12k; LCSC C11702 -> C25752
- R328: renamed from TP302; value BCK -> 1k; footprint TestPoint:TestPoint_Pad_D1.0mm -> Resistor_SMD:R_1206_3216Metric; symbol Connector:TestPoint -> Device:R_Small; JLC bare pad -> Basic; LCSC (none) -> C4410; Note (none) -> 1206: survives output-to-output patching; Tolerance (none) -> 1%; now in the parts list
- U302: renamed from R308; value 1M -> TL074HIDR; footprint Resistor_SMD:R_0402_1005Metric -> Package_SO:SOIC-14_3.9x8.7mm_P1.27mm; symbol Device:R_Small -> Amplifier_Operational:TL074; JLC Basic -> Extended; LCSC C26083 -> C2878713; MPN (none) -> TL074HIDR; Note holds the jack side at 0 V -> (none); Tolerance 1% -> (none)
Connections:
- net +12V: now also C319.1; no longer R322.1
- net +3V3D: now also R305.1; no longer C303.1, C304.1, U301.7 (V_{DD})
- net +5VA: now also D301.2 (K), FB301.1; no longer C301.1, C302.1, U301.24 (V_{CC})
- net -12V: now also C320.1; no longer C316.1
- net AIN1: now also R309.1; no longer U302.1
- net AIN2: now also R313.1, C311.1; no longer D301.1, R312.1
- net AOUT1: now also R321.2
- net AOUT2: now also R328.2; no longer R323.2
- net BCK: now also TP302.1; no longer R328.1
- net CODEC_MODE: now also R306.1; no longer R305.1
- net CODEC_RST: now also R305.2, J303.1 (Pin_1); no longer R304.2
- net GND: now also C309.2, C312.2, D301.1 (A), R306.2, R313.2, R320.2, C317.2, C319.2, C320.2, J303.2 (Pin_2), R309.2, R327.2; no longer C313.2, C316.2, R305.2, R312.2, R322.2, U302.2
- net VCOM: now also C309.1, C312.1, U302.3 (+)
- net VINL: now also D301.3 (COM), R310.2; no longer C307.2
- net VINR: now also R314.2; no longer R313.2
- net VOUTL_P: now also R316.1; no longer R314.1
- net VOUTR_N: now also R322.1; no longer R319.1
- net VOUTR_P: now also R323.1; no longer R320.1
- net at R311.1: now also R312.2, U302.6 (-), C310.1; no longer D301.2
- net at U302.8: now also C313.2, R319.2, R321.1; no longer C312.2
- net at C307.1: now also R307.1, U302.2 (-), R308.2; no longer R306.2
- net at U302.10 (+): now also C314.1, R318.2; no longer R314.2
- net at R307.2: now also C307.2, R310.1, U302.1; no longer R306.1
- net at C308.2: now also R308.1; no longer R307.1
- new net: C315.2, R316.2, R318.1, R320.1
- new net: C318.2, R323.2, R325.1, R327.1
- new net: C318.1, R322.2, R324.1, R326.1
- new net: C316.2, R326.2, R328.1, U302.14
- new net: C317.1, R325.2, U302.12 (+)
- new net: C316.1, R324.2, U302.13 (-)
- new net: C313.1, R317.2, U302.9 (-)
- new net: C315.1, R315.2, R317.1, R319.1
- new net: C310.2, R311.2, R314.1, U302.7
- new net: C311.2, R312.1
- new net CODEC_VCC: C301.1, C302.1, FB301.2, U301.24 (V_{CC})
- new net CODEC_VDD: C303.1, C304.1, R304.2, U301.7 (V_{DD})
Other:
- note added: "AUDIO INPUTS: 22 Vpp → 3 Vpp (codec full scale). AC-coupled, inverting (firmware flips the sign). ±12 V stays inside the codec rails, so the BAT54S clamps only act on faults. 100 nF on each + input decouples VCOM (12.5 kΩ source) at the op-amp, as the Patch SM does."
- note added: "AUDIO OUTPUTS: balanced second-order MFB low-pass (Beads' topology), gain 30k/12k = 2.5, so 8 Vpp → 20 Vpp, DC-coupled, non-inverting (VOUT+ to the + side). 1 nF C0G across the two nodes and 100 pF from each op-amp input: f0 ≈ 65 kHz, Q ≈ 0.73, flat to 20 kHz (Basic parts except the 1 nF C0G). 1 kΩ 1206 out survives output-to-output patching."
- note added: "PCM3060 in hardware-control mode, the same straps as Mutable Beads: MODE 220 kΩ to DGND = parallel control with differential outputs; FMT low = 24-bit I2S, IFMD low = ADC and DAC both slaves, DEMP low = no de-emphasis. One I2S bus feeds both halves. RST is pulled up, so the codec starts by itself; CODEC_RST also reaches a hole (J303) so firmware can hold it in reset, as Beads does. Full scale is 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"
- note removed: "AUDIO INPUTS: 10 Vpp → 3 Vpp. AC-coupled, inverting (firmware flips the sign), ±12 V tolerant. The 1 kΩ into the codec's 10 kΩ input sets part of the gain; BAT54S clamps to the codec rails."
- note removed: "AUDIO OUTPUTS: difference amplifier, gain 15k/12k = 1.25, so 8 Vpp → 10 Vpp (±5 V), DC-coupled. 100 pF C0G across each 15 kΩ: a pole at 106 kHz on top of the codec's own RC filter."
- note removed: "PCM3060 in hardware-control mode: MODE 220 kΩ to DGND = parallel control with differential outputs; FMT low = 24-bit I2S, IFMD low = ADC and DAC both slaves, DEMP low = no de-emphasis. One I2S bus feeds both halves (SCKI1/2, BCK1/2, LRCK1/2 joined). RST is pulled up, so the codec starts by itself 1024 clocks after power-up. ADC full scale 0.6 × VCC = 3 Vpp around VCOM; DAC 8 Vpp differential."
- moved on the sheet: C312, C314, R314, R317, R319, R320

Commit message: Analogue board: checkpoint 3 started; double-sided, floorplan placed
- pcb.py generates analogue_board.kicad_pcb from the netlist: outline,
  JLC 4-layer stack-up, every footprint with nets and schematic links
  (KiCad schematic parity: 0 differences), parked parts beside the board,
  courtyard area budget, DRC and 3D renders of both faces.
- Area budget: the courtyards need 104% of one face before routing, so
  David chose double-sided assembly (JLC Standard PCBA, about $100 more
  per order, to confirm on a quote).
- Floorplan in placement.py: analogue ICs at the top under the modules,
  furthest from the buck; logic below; power bottom right around J201;
  MIDI bottom left; 99 wiring-field holes in three columns lined up with
  the edge-strip positions, each group beside its circuit.
- Library: module socket courtyards cover only their header rows; the
  wiring holes get their own footprint with a one-pitch courtyard.
- Spec records the decision, the floorplan and David's answers: 11 mm to
  the deck in 10HP (deck parts 2 mm at most); holes tinned both faces.

Co-Authored-By: Claude Opus 5.5 <noreply@anthropic.com>
Parts:
- J301, J302: footprint Connector_PinHeader_2.54mm:PinHeader_1x03_P2.54mm_Vertical -> analogue_board:WiringHoles_1x03
- J303: footprint Connector_PinHeader_2.54mm:PinHeader_1x02_P2.54mm_Vertical -> analogue_board:WiringHoles_1x02
Changed lines of the file:
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@@
 			)
 		)
-		(property "Footprint" "Connector_PinHeader_2.54mm:PinHeader_1x02_P2.54mm_Vertical"
+		(property "Footprint" "analogue_board:WiringHoles_1x02"
 			(at 76.2 203.2 0)
 			(effects
@@
 			)
 		)
-		(property "Footprint" "Connector_PinHeader_2.54mm:PinHeader_1x03_P2.54mm_Vertical"
+		(property "Footprint" "analogue_board:WiringHoles_1x03"
 			(at 340.36 66.04 0)
 			(effects
@@
 			)
 		)
-		(property "Footprint" "Connector_PinHeader_2.54mm:PinHeader_1x03_P2.54mm_Vertical"
+		(property "Footprint" "analogue_board:WiringHoles_1x03"
 			(at 340.36 177.8 0)
 			(effects

Commit message: Analogue board: first-pass placement; space reclaimed; four wiring banks
- autoplace.py places every unanchored part as close as it fits to the
  pins it connects to: decoupling capacitors at their pin, chains growing
  from their ICs, the buck's loop kept on one face. All 430 parts placed;
  DRC courtyards clean, schematic parity clean, heights checked (<= 2.5 mm
  under the modules, <= 8 mm in the USB keep-outs).
- Space reclaimed (David): Teensy socket without holes for its unused
  far-end pins 20-28 (headers 1x19 + 1x20); right strip (10HP only) without
  holes at 11-15 and 26-30, and outer hole only at 10, 16, 31. checks.py
  lets a project footprint omit only pins the netlist leaves unconnected.
- 74HCT595 in TSSOP-16 (74HCT595PW, C99710, same pinout) sideways in the
  right channel; vertical Qwiic socket (BM04B-SRSS-TB, C160390) below the
  modules, its cable straight up (the side-entry plug had no clear run).
- Wiring field as four mixed banks (David): each quarter of the board has
  some of every channel type, 50/50 left and right, jack-detect holes
  beside their inputs; wiring.py holds the plan, schematic and placement
  both read it. 94 holes.
- Reference designators off the silkscreen for passives and hole groups.

Co-Authored-By: Claude Opus 5.5 <noreply@anthropic.com>
Parts:
- removed J302: Audio out holes, analogue_board:WiringHoles_1x03, symbol Connector_Generic:Conn_01x03
- added J311: Holes, left bottom, analogue_board:WiringHoles_1x01, symbol Connector_Generic:Conn_01x01
- added J312: Holes, right top, analogue_board:WiringHoles_1x01, symbol Connector_Generic:Conn_01x01
- added J313: Holes, right middle, analogue_board:WiringHoles_1x01, symbol Connector_Generic:Conn_01x01
- J310: renamed from J301; value Audio in holes -> Holes, left top; footprint analogue_board:WiringHoles_1x03 -> analogue_board:WiringHoles_1x01; symbol Connector_Generic:Conn_01x03 -> Connector_Generic:Conn_01x01
Connections:
- net AIN2: now also J312.1 (Pin_1); no longer J310.2 (Pin_2)
- net AOUT1: now also J311.1 (Pin_1)
- net AOUT2: now also J313.1 (Pin_1)
- net GND: no longer J310.3 (Pin_3)
Changed lines of the file:
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@@
 	)
 	(symbol
-		(lib_id "Connector_Generic:Conn_01x03")
-		(at 340.36 66.04 0)
+		(lib_id "Connector_Generic:Conn_01x01")
+		(at 340.36 60.96 0)
 		(unit 1)
 		(exclude_from_sim no)
@@
 		(on_board yes)
 		(dnp no)
-		(property "Reference" "J301"
+		(property "Reference" "J310"
+			(at 340.36 58.42 0)
+			(effects
+				(font (size 1.27 1.27))
+			)
+		)
+		(property "Value" "Holes, left top"
+			(at 340.36 63.5 0)
+			(effects
+				(font (size 1.27 1.27))
+			)
+		)
+		(property "Footprint" "analogue_board:WiringHoles_1x01"
 			(at 340.36 60.96 0)
 			(effects
 				(font (size 1.27 1.27))
-			)
-		)
-		(property "Value" "Audio in holes"
-			(at 340.36 71.12 0)
-			(effects
-				(font (size 1.27 1.27))
-			)
-		)
-		(property "Footprint" "analogue_board:WiringHoles_1x03"
-			(at 340.36 66.04 0)
-			(effects
-				(font (size 1.27 1.27))
 				(hide yes)
 			)
 		)
 		(property "Datasheet" ""
-			(at 340.36 66.04 0)
+			(at 340.36 60.96 0)
 			(effects
 				(font (size 1.27 1.27))
@@
 		)
 		(property "Description" ""
-			(at 340.36 66.04 0)
+			(at 340.36 60.96 0)
 			(effects
 				(font (size 1.27 1.27))
@@
 		)
 		(property "JLC" "bare holes"
-			(at 340.36 66.04 0)
+			(at 340.36 60.96 0)
 			(effects
 				(font (size 1.27 1.27))
@@
 		)
 		(pin "1"
-		)
-		(pin "2"
-		)
-		(pin "3"
 		)
 		(instances
 			(project "analogue_board"
 				(path "/e6cfe5fb-cd34-5945-b37d-aca61e0551b2/47430451-5b2e-5bac-802f-17f0b1d5ba28"
-					(reference "J301")
+					(reference "J310")
 					(unit 1)
 				)
@@
 	)
 	(label "AIN1"
-		(at 332.74 63.5 180)
+		(at 332.74 60.96 180)
 		(effects
 			(font (size 1.27 1.27))
@@
 		)
 	)
-	(label "AIN2"
-		(at 332.74 66.04 180)
-		(effects
-			(font (size 1.27 1.27))
-			(justify right bottom)
-		)
-	)
 	(symbol
-		(lib_id "power:GND")
-		(at 332.74 68.58 270)
-		(unit 1)
-		(exclude_from_sim no)
-		(in_bom yes)
-		(on_board yes)
-		(dnp no)
-		(property "Reference" "#PWR113"
-			(at 326.39 68.58 90)
-			(effects
-				(font (size 1.27 1.27))
-				(hide yes)
-			)
-		)
-		(property "Value" "GND"
-			(at 328.93 68.58 90)
-			(effects
-				(font (size 1.27 1.27))
-				(justify right)
-			)
-		)
-		(property "Footprint" ""
-			(at 332.74 68.58 90)
-			(effects
-				(font (size 1.27 1.27))
-				(hide yes)
-			)
-		)
-		(property "Datasheet" ""
-			(at 332.74 68.58 90)
-			(effects
-				(font (size 1.27 1.27))
-				(hide yes)
-			)
-		)
-		(property "Description" ""
-			(at 332.74 68.58 90)
-			(effects
-				(font (size 1.27 1.27))
-				(hide yes)
-			)
-		)
-		(pin "1"
-		)
-		(instances
-			(project "analogue_board"
-				(path "/e6cfe5fb-cd34-5945-b37d-aca61e0551b2/47430451-5b2e-5bac-802f-17f0b1d5ba28"
-					(reference "#PWR113")
-					(unit 1)
-				)
-			)
-		)
-	)
-	(symbol
-		(lib_id "Connector_Generic:Conn_01x03")
-		(at 340.36 177.8 0)
+		(lib_id "Connector_Generic:Conn_01x01")
+		(at 340.36 71.12 0)
 		(unit 1)
 		(exclude_from_sim no)
@@
 		(on_board yes)
 		(dnp no)
-		(property "Reference" "J302"
-			(at 340.36 172.72 0)
-			(effects
-				(font (size 1.27 1.27))
-			)
-		)
-		(property "Value" "Audio out holes"
-			(at 340.36 182.88 0)
-			(effects
-				(font (size 1.27 1.27))
-			)
-		)
-		(property "Footprint" "analogue_board:WiringHoles_1x03"
-			(at 340.36 177.8 0)
+		(property "Reference" "J311"
+			(at 340.36 68.58 0)
+			(effects
+				(font (size 1.27 1.27))
+			)
+		)
+		(property "Value" "Holes, left bottom"
+			(at 340.36 73.66 0)
+			(effects
+				(font (size 1.27 1.27))
+			)
+		)
+		(property "Footprint" "analogue_board:WiringHoles_1x01"
+			(at 340.36 71.12 0)
 			(effects
 				(font (size 1.27 1.27))
@@
 		)
 		(property "Datasheet" ""
-			(at 340.36 177.8 0)
+			(at 340.36 71.12 0)
 			(effects
 				(font (size 1.27 1.27))
@@
 		)
 		(property "Description" ""
-			(at 340.36 177.8 0)
+			(at 340.36 71.12 0)
 			(effects
 				(font (size 1.27 1.27))
@@
 		)
 		(property "JLC" "bare holes"
-			(at 340.36 177.8 0)
+			(at 340.36 71.12 0)
 			(effects
 				(font (size 1.27 1.27))
@@
 		)
 		(pin "1"
-		)
-		(pin "2"
-		)
-		(pin "3"
 		)
 		(instances
 			(project "analogue_board"
 				(path "/e6cfe5fb-cd34-5945-b37d-aca61e0551b2/47430451-5b2e-5bac-802f-17f0b1d5ba28"
-					(reference "J302")
+					(reference "J311")
 					(unit 1)
 				)
@@
 	)
 	(label "AOUT1"
-		(at 332.74 175.26 180)
+		(at 332.74 71.12 180)
 		(effects
 			(font (size 1.27 1.27))
@@
 		)
 	)
-	(label "AOUT2"
-		(at 332.74 177.8 180)
+	(symbol
+		(lib_id "Connector_Generic:Conn_01x01")
+		(at 340.36 81.28 0)
+		(unit 1)
+		(exclude_from_sim no)
+		(in_bom no)
+		(on_board yes)
+		(dnp no)
+		(property "Reference" "J312"
+			(at 340.36 78.74 0)
+			(effects
+				(font (size 1.27 1.27))
+			)
+		)
+		(property "Value" "Holes, right top"
+			(at 340.36 83.82 0)
+			(effects
+				(font (size 1.27 1.27))
+			)
+		)
+		(property "Footprint" "analogue_board:WiringHoles_1x01"
+			(at 340.36 81.28 0)
+			(effects
+				(font (size 1.27 1.27))
+				(hide yes)
+			)
+		)
+		(property "Datasheet" ""
+			(at 340.36 81.28 0)
+			(effects
+				(font (size 1.27 1.27))
+				(hide yes)
+			)
+		)
+		(property "Description" ""
+			(at 340.36 81.28 0)
+			(effects
+				(font (size 1.27 1.27))
+				(hide yes)
+			)
+		)
+		(property "JLC" "bare holes"
+			(at 340.36 81.28 0)
+			(effects
+				(font (size 1.27 1.27))
+				(hide yes)
+			)
+		)
+		(pin "1"
+		)
+		(instances
+			(project "analogue_board"
+				(path "/e6cfe5fb-cd34-5945-b37d-aca61e0551b2/47430451-5b2e-5bac-802f-17f0b1d5ba28"
+					(reference "J312")
+					(unit 1)
+				)
+			)
+		)
+	)
+	(label "AIN2"
+		(at 332.74 81.28 180)
 		(effects
 			(font (size 1.27 1.27))
@@
 	)
 	(symbol
-		(lib_id "power:GND")
-		(at 332.74 180.34 270)
+		(lib_id "Connector_Generic:Conn_01x01")
+		(at 340.36 91.44 0)
 		(unit 1)
 		(exclude_from_sim no)
-		(in_bom yes)
+		(in_bom no)
 		(on_board yes)
 		(dnp no)
-		(property "Reference" "#PWR114"
-			(at 326.39 180.34 90)
-			(effects
-				(font (size 1.27 1.27))
-				(hide yes)
-			)
-		)
-		(property "Value" "GND"
-			(at 328.93 180.34 90)
-			(effects
-				(font (size 1.27 1.27))
-				(justify right)
-			)
-		)
-		(property "Footprint" ""
-			(at 332.74 180.34 90)
+		(property "Reference" "J313"
+			(at 340.36 88.9 0)
+			(effects
+				(font (size 1.27 1.27))
+			)
+		)
+		(property "Value" "Holes, right middle"
+			(at 340.36 93.98 0)
+			(effects
+				(font (size 1.27 1.27))
+			)
+		)
+		(property "Footprint" "analogue_board:WiringHoles_1x01"
+			(at 340.36 91.44 0)
 			(effects
 				(font (size 1.27 1.27))
@@
 		)
 		(property "Datasheet" ""
-			(at 332.74 180.34 90)
+			(at 340.36 91.44 0)
 			(effects
 				(font (size 1.27 1.27))
@@
 		)
 		(property "Description" ""
-			(at 332.74 180.34 90)
+			(at 340.36 91.44 0)
+			(effects
+				(font (size 1.27 1.27))
+				(hide yes)
+			)
+		)
+		(property "JLC" "bare holes"
+			(at 340.36 91.44 0)
 			(effects
 				(font (size 1.27 1.27))
@@
 			(project "analogue_board"
 				(path "/e6cfe5fb-cd34-5945-b37d-aca61e0551b2/47430451-5b2e-5bac-802f-17f0b1d5ba28"
-					(reference "#PWR114")
+					(reference "J313")
 					(unit 1)
 				)
 			)
+		)
+	)
+	(label "AOUT2"
+		(at 332.74 91.44 180)
+		(effects
+			(font (size 1.27 1.27))
+			(justify right bottom)
 		)
 	)
@@
 	)
 	(wire
-		(pts (xy 332.74 63.5) (xy 335.28 63.5))
-		(stroke (width 0) (type default))
-	)
-	(wire
-		(pts (xy 332.74 66.04) (xy 335.28 66.04))
-		(stroke (width 0) (type default))
-	)
-	(wire
-		(pts (xy 332.74 68.58) (xy 335.28 68.58))
-		(stroke (width 0) (type default))
-	)
-	(wire
-		(pts (xy 332.74 175.26) (xy 335.28 175.26))
-		(stroke (width 0) (type default))
-	)
-	(wire
-		(pts (xy 332.74 177.8) (xy 335.28 177.8))
-		(stroke (width 0) (type default))
-	)
-	(wire
-		(pts (xy 332.74 180.34) (xy 335.28 180.34))
-		(stroke (width 0) (type default))
-	)
+		(pts (xy 332.74 60.96) (xy 335.28 60.96))
+		(stroke (width 0) (type default))
+	)
+	(wire
+		(pts (xy 332.74 71.12) (xy 335.28 71.12))
+		(stroke (width 0) (type default))
+	)
+	(wire
+		(pts (xy 332.74 81.28) (xy 335.28 81.28))
+		(stroke (width 0) (type default))
+	)
+	(wire
+		(pts (xy 332.74 91.44) (xy 335.28 91.44))
+		(stroke (width 0) (type default))
+	)
