File: hardware/analogue_board/teensy_core_midi/routed_trial/analogue_board_teensy_core_midi_routed.kicad_pcb (KiCad board)
At the start: 6 copper layers, 49.6 x 103 mm, 368 parts, among them J1001 TRS MIDI holes, J101 Spare GPIO, MIDI links, J201 Eurorack power 2x5 shrouded, J303 Codec RST, J310 Holes, left top, J311 Holes, left bottom, J312 Holes, right top, J313 Holes, right middle, J410 Holes, left top, J411 Holes, left bottom, J412 Holes, left top, J413 Holes, right top, J414 Holes, right middle, J603 Gate expansion: QH', SRCLK, R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, J610 Holes, left top, J611 Holes, left bottom, J612 Holes, left top, J613 Holes, left bottom, J614 Holes, right top, J615 Holes, right middle, J703 I2C holes for a wired display, J704 WS2812 chain holes, J710 Holes, left top, J711 Holes, left bottom, J712 Holes, left top, J713 Holes, left bottom, J714 Holes, right top, J715 Holes, right middle, J716 Holes, right top, J810 Holes, left top, J811 Holes, left bottom, J812 Holes, right top, J813 Holes, right middle, J901 Edge strip, left, J902 Edge strip, right, U1001 SN74AHCT1G125DBVR, U1002 H11L1SR2M, U201 TPS54308DDCR, U202 L78M05ABDT-TR, U203 XC6206P332MR-G, U204 XC6206P332MR-G, U301 PCM3060PWR, U302 TL074HIDR, U401 ADS8688IDBTR, U402 DG412DQ-T1-E3, U403 DG412DQ-T1-E3, U501 DAC8568IAPWR, U502 TL074HIDR, U504 TL074HIDR, U601 MCP3208-CI/SL, U602 74HCT595PW, U701 TCA9555PWR, U702 M24C64-RMN6TP, U703 SN74AHCT1G125DBVR, U801 LM393DR2G, U802 LM393DR2G

Commit message: Analogue board: Teensy core board labelled, order files for JLCPCB
- labels.py: block numbers (W1, W2 ...) beside the wiring blocks and names beside the test
  points, on both faces where they fit; output/wiring_map.md lists every block's holes and
  signals and every test point, with 1:1 PDFs of each face to print
- fab.py run on the routed board: teensy_core_midi/fab/ holds the Gerber zip, JLC BOM and CPL
  (300 placements, 59 part types); the loose Gerbers are ignored
- finish.py: a closing step adds a direct capacitor-to-pin track where the routed one is over
  4 mm (crossing other nets if need be, never another reference capacitor's); ground vias
  joined only to the plane are removed; whatever KiCad's DRC calls a dead end is taken up
- The four decoupling paths still over 4 mm (REFIO 9.2, U402 -12 V 5.8, POT_REF 4.7, U202
  input 4.3 mm) are accepted for Rev A (David); the SMA diode notice is benign

Co-Authored-By: Claude Opus 5.5 <noreply@anthropic.com>
Other:
- board text added: "+12V"
- board text added: "+3V3D"
- board text added: "+5VD"
- board text added: "-12V"
- board text added: "5V MOD"
- board text added: "B MISO"
- board text added: "CS 595"
- board text added: "CS ADC"
- board text added: "DIN"
- board text added: "DOUT"
- board text added: "GND"
- board text added: "INT"
- board text added: "SCL"
- board text added: "SDA"
- board text added: "W1"
- board text added: "W2"
- board text added: "W3"
- board text added: "W4"
- board text added: "W5"
- board text added: "W6"
- board text added: "W7"
- board text added: "W9"
