File: hardware/analogue_board/pico_core_midi/analogue_board_pico_core_midi.kicad_pcb (KiCad board)
At the start: 4 copper layers, 49.6 x 103 mm, 371 parts, among them J1001 TRS MIDI holes, J101 Spare GPIO, MIDI links, RUN, J201 Eurorack power 2x5 shrouded, J303 Codec RST, J310 Holes, left top, J311 Holes, left bottom, J312 Holes, right top, J313 Holes, right middle, J410 Holes, left top, J411 Holes, left bottom, J412 Holes, left top, J413 Holes, right top, J414 Holes, right middle, J603 Gate expansion: QH', SRCLK, R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, J610 Holes, left top, J611 Holes, left bottom, J612 Holes, left top, J613 Holes, left bottom, J614 Holes, right top, J615 Holes, right middle, J703 I2C holes for a wired display, J704 WS2812 chain holes, J710 Holes, left top, J711 Holes, left bottom, J712 Holes, left top, J713 Holes, left bottom, J714 Holes, right top, J715 Holes, right middle, J810 Holes, left top, J811 Holes, left bottom, J812 Holes, right top, J813 Holes, right middle, J901 Edge strip, left, J902 Edge strip, right, Q201 AO3401A, U1001 SN74AHCT1G125DBVR, U1002 H11L1SR2M, U201 TPS54308DDCR, U202 L78M05ABDT-TR, U203 XC6206P332MR-G, U204 XC6206P332MR-G, U301 PCM3060PWR, U302 TL074HIDR, U401 ADS8688IDBTR, U402 DG412DQ-T1-E3, U403 DG412DQ-T1-E3, U501 DAC8568IAPWR, U502 TL074HIDR, U504 TL074HIDR, U601 MCP3208-CI/SL, U602 74HCT595PW, U701 TCA9555PWR, U702 M24C64-RMN6TP, U703 SN74AHCT1G125DBVR, U801 LM393DR2G, U802 LM393DR2G

Commit message: Analogue board: the Pico board routes completely
pico_core_midi (Pico 2 / ESP32-P4, the core set with MIDI) routes with no unconnected item
and no copper fault, and every IC supply pin within 4 mm of its capacitor. Routed board in
pico_core_midi/routed_trial/, labels and wiring map, JLC files in pico_core_midi/fab/. Held:
David orders it after the Teensy board's bring-up.

What got it there:
- David's re-laid top: no chip over another on the opposite face (ADC lowered, DAC and CV
  op-amp turned and stacked, DG412s and U504 where nothing is above them, U203 moved out);
  the right-top wiring bank into the right strip's gap; no bus test points; U204 out from
  under the module
- autoroute.py --plane=+5VD: a +5VD plane on In4 whose pads get their own vias before routing
  (stage 1 left 14 instead of 35)
- finish.py: escape lanes kept clear of pre-route ground vias (ADC pin 2 had been fenced in by
  six); decoupling tracks protected from rip-up; plane nets handled throughout
- finish.py fixes: an empty route that looped for hours (no empty routes, a no-progress
  guard); row-at-a-time marking and A* search; KiCad's own dead ends removed

Journal, README and spec updated with the result.

Co-Authored-By: Claude Opus 5.5 <noreply@anthropic.com>
Parts:
- removed TP301: MCLK, TestPoint:TestPoint_Pad_D1.0mm
- removed TP302: BCK, TestPoint:TestPoint_Pad_D1.0mm
- removed TP303: LRCK, TestPoint:TestPoint_Pad_D1.0mm
- removed TP304: I2S_DOUT, TestPoint:TestPoint_Pad_D1.0mm
- removed TP305: I2S_DIN, TestPoint:TestPoint_Pad_D1.0mm
- removed TP401: SPIA_SCK, TestPoint:TestPoint_Pad_D1.0mm
- removed TP402: SPIA_MOSI, TestPoint:TestPoint_Pad_D1.0mm
- removed TP403: SPIA_MISO, TestPoint:TestPoint_Pad_D1.0mm
- removed TP404: CS_ADC, TestPoint:TestPoint_Pad_D1.0mm
- removed TP405: CS_DAC, TestPoint:TestPoint_Pad_D1.0mm
- removed TP601: SPIB_SCK, TestPoint:TestPoint_Pad_D1.0mm
- removed TP602: SPIB_MOSI, TestPoint:TestPoint_Pad_D1.0mm
- removed TP603: SPIB_MISO, TestPoint:TestPoint_Pad_D1.0mm
- removed TP604: CS_595, TestPoint:TestPoint_Pad_D1.0mm
- removed TP605: CS_POT, TestPoint:TestPoint_Pad_D1.0mm
- removed TP701: SDA, TestPoint:TestPoint_Pad_D1.0mm
- removed TP702: SCL, TestPoint:TestPoint_Pad_D1.0mm
- removed TP703: EXP_INT, TestPoint:TestPoint_Pad_D1.0mm
- added J616: Holes, right top, analogue_board:WiringHoles_1x02, F.Cu at (77.7, 57.5)
- C218, C405, C408, C415, C416, C418, C419, C505, C506, C510, C513, C605, C606, C610, C706, D302, D601, R209, R306, R315, R327, R404, R405, R413, R423, R426, R506, R508, R509, R510, R511, R512, R515, R603, R604, R605, R606, R715, R717, R719, R806, TP202, TP205, TP207, TP208: moved to F.Cu
- C220, C308, C311, C315, C403, C404, C412, C413, C420, C501, C504, C507, C511, C512, C608, C707, C709, D301, D406, D603, R1008, R210, R301, R308, R313, R322, R408, R409, R416, R501, R502, R503, R507, R514, R609, R610, R612, R619, R701, R707, R709, R711, R712, R713: moved to B.Cu
- J312, J413, J714, J812: value Holes, right top -> Holes, right middle
- J313, J414, J715, J813: value Holes, right middle -> Holes, right top
- J614: value Holes, right top -> Holes, right middle; footprint analogue_board:WiringHoles_1x04 -> analogue_board:WiringHoles_1x01
- J615: value Holes, right middle -> Holes, right top; footprint analogue_board:WiringHoles_1x01 -> analogue_board:WiringHoles_1x02
- moved J614 48.3 mm to (72.6, 90.5)
- moved J312 40.6 mm to (72.6, 77.8)
- moved J714 40.6 mm to (72.6, 93.0)
- moved J812 40.6 mm to (72.6, 80.3)
- moved J413 40.6 mm to (72.6, 72.7)
- moved J715 30.9 mm to (77.7, 62.5)
- moved J615 25.5 mm to (75.1, 65.1)
- moved C501 20.2 mm to (64.5, 49.7)
- moved C420 19.2 mm to (52.0, 51.2), turned to 90 degrees
- moved C418 19.2 mm to (50.1, 51.8), turned to 0 degrees
- moved C513 18.9 mm to (54.5, 50.5)
- moved D404 18.7 mm to (67.7, 51.9), turned to 90 degrees
- moved D402 18.3 mm to (45.8, 32.1)
- moved R313 18.2 mm to (67.5, 62.6)
- moved J313 18.0 mm to (75.1, 60.0)
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Connections:
- J312 pad 1: /Codec & audio/AIN2 -> /Codec & audio/AOUT2
- J313 pad 1: /Codec & audio/AOUT2 -> /Codec & audio/AIN2
- J413 pad 1: /CV jacks & ADC/CV4 -> /CV jacks & ADC/CV6
- J414 pad 1: /CV jacks & ADC/CV6 -> /CV jacks & ADC/CV4
- J614 pad 1: /Pots & gate outs/POT5 -> /Pots & gate outs/GOUT4
- J615 pad 1: /Pots & gate outs/GOUT4 -> /Pots & gate outs/POT5
- J714 pad 1: /Expander, I2C & LEDs/SW6 -> /Expander, I2C & LEDs/SW8
- J714 pad 2: /Expander, I2C & LEDs/SW7 -> /Expander, I2C & LEDs/SW9
- J715 pad 1: /Expander, I2C & LEDs/SW8 -> /Expander, I2C & LEDs/SW6
- J715 pad 2: /Expander, I2C & LEDs/SW9 -> /Expander, I2C & LEDs/SW7
- J812 pad 1: /Gate ins/GIN3 -> /Gate ins/GIN4
- J813 pad 1: /Gate ins/GIN4 -> /Gate ins/GIN3
