File: hardware/analogue_board/pico_core_midi/codec_audio.kicad_sch (KiCad schematic)
At the start: 63 parts, among them J303 Codec RST, J310 Holes, left top, J311 Holes, left bottom, J312 Holes, right top, J313 Holes, right middle, U301 PCM3060PWR, U302 TL074HIDR

Commit message: Analogue board: the Pico board routes completely
pico_core_midi (Pico 2 / ESP32-P4, the core set with MIDI) routes with no unconnected item
and no copper fault, and every IC supply pin within 4 mm of its capacitor. Routed board in
pico_core_midi/routed_trial/, labels and wiring map, JLC files in pico_core_midi/fab/. Held:
David orders it after the Teensy board's bring-up.

What got it there:
- David's re-laid top: no chip over another on the opposite face (ADC lowered, DAC and CV
  op-amp turned and stacked, DG412s and U504 where nothing is above them, U203 moved out);
  the right-top wiring bank into the right strip's gap; no bus test points; U204 out from
  under the module
- autoroute.py --plane=+5VD: a +5VD plane on In4 whose pads get their own vias before routing
  (stage 1 left 14 instead of 35)
- finish.py: escape lanes kept clear of pre-route ground vias (ADC pin 2 had been fenced in by
  six); decoupling tracks protected from rip-up; plane nets handled throughout
- finish.py fixes: an empty route that looped for hours (no empty routes, a no-progress
  guard); row-at-a-time marking and A* search; KiCad's own dead ends removed

Journal, README and spec updated with the result.

Co-Authored-By: Claude Opus 5.5 <noreply@anthropic.com>
Parts:
- removed TP301: MCLK, TestPoint:TestPoint_Pad_D1.0mm, symbol Connector:TestPoint
- removed TP302: BCK, TestPoint:TestPoint_Pad_D1.0mm, symbol Connector:TestPoint
- removed TP303: LRCK, TestPoint:TestPoint_Pad_D1.0mm, symbol Connector:TestPoint
- removed TP304: I2S_DOUT, TestPoint:TestPoint_Pad_D1.0mm, symbol Connector:TestPoint
- removed TP305: I2S_DIN, TestPoint:TestPoint_Pad_D1.0mm, symbol Connector:TestPoint
- J312: value Holes, right top -> Holes, right middle
- J313: value Holes, right middle -> Holes, right top
Connections:
- net AIN2: now also J313.1 (Pin_1); no longer J312.1 (Pin_1)
- net AOUT2: now also J312.1 (Pin_1); no longer J313.1 (Pin_1)
