File: hardware/analogue_board/pico_core_midi/cv_io.kicad_sch (KiCad schematic)
At the start: 66 parts, among them J410 Holes, left top, J411 Holes, left bottom, J412 Holes, left top, J413 Holes, right top, J414 Holes, right middle, U401 ADS8688IDBTR, U402 DG412DQ-T1-E3, U403 DG412DQ-T1-E3

Commit message: Analogue board: the Pico board routes completely
pico_core_midi (Pico 2 / ESP32-P4, the core set with MIDI) routes with no unconnected item
and no copper fault, and every IC supply pin within 4 mm of its capacitor. Routed board in
pico_core_midi/routed_trial/, labels and wiring map, JLC files in pico_core_midi/fab/. Held:
David orders it after the Teensy board's bring-up.

What got it there:
- David's re-laid top: no chip over another on the opposite face (ADC lowered, DAC and CV
  op-amp turned and stacked, DG412s and U504 where nothing is above them, U203 moved out);
  the right-top wiring bank into the right strip's gap; no bus test points; U204 out from
  under the module
- autoroute.py --plane=+5VD: a +5VD plane on In4 whose pads get their own vias before routing
  (stage 1 left 14 instead of 35)
- finish.py: escape lanes kept clear of pre-route ground vias (ADC pin 2 had been fenced in by
  six); decoupling tracks protected from rip-up; plane nets handled throughout
- finish.py fixes: an empty route that looped for hours (no empty routes, a no-progress
  guard); row-at-a-time marking and A* search; KiCad's own dead ends removed

Journal, README and spec updated with the result.

Co-Authored-By: Claude Opus 5.5 <noreply@anthropic.com>
Parts:
- removed TP401: SPIA_SCK, TestPoint:TestPoint_Pad_D1.0mm, symbol Connector:TestPoint
- removed TP402: SPIA_MOSI, TestPoint:TestPoint_Pad_D1.0mm, symbol Connector:TestPoint
- removed TP403: SPIA_MISO, TestPoint:TestPoint_Pad_D1.0mm, symbol Connector:TestPoint
- removed TP404: CS_ADC, TestPoint:TestPoint_Pad_D1.0mm, symbol Connector:TestPoint
- removed TP405: CS_DAC, TestPoint:TestPoint_Pad_D1.0mm, symbol Connector:TestPoint
- J413: value Holes, right top -> Holes, right middle
- J414: value Holes, right middle -> Holes, right top
Connections:
- net CV4: now also J414.1 (Pin_1); no longer J413.1 (Pin_1)
- net CV6: now also J413.1 (Pin_1); no longer J414.1 (Pin_1)
