File: hardware/analogue_board/pico_core_midi/expander_i2c.kicad_sch (KiCad schematic)
At the start: 49 parts, among them J703 I2C holes for a wired display, J704 WS2812 chain holes, J710 Holes, left top, J711 Holes, left bottom, J712 Holes, left top, J713 Holes, left bottom, J714 Holes, right top, J715 Holes, right middle, U701 TCA9555PWR, U702 M24C64-RMN6TP, U703 SN74AHCT1G125DBVR

Commit message: Analogue board: the Pico board routes completely
pico_core_midi (Pico 2 / ESP32-P4, the core set with MIDI) routes with no unconnected item
and no copper fault, and every IC supply pin within 4 mm of its capacitor. Routed board in
pico_core_midi/routed_trial/, labels and wiring map, JLC files in pico_core_midi/fab/. Held:
David orders it after the Teensy board's bring-up.

What got it there:
- David's re-laid top: no chip over another on the opposite face (ADC lowered, DAC and CV
  op-amp turned and stacked, DG412s and U504 where nothing is above them, U203 moved out);
  the right-top wiring bank into the right strip's gap; no bus test points; U204 out from
  under the module
- autoroute.py --plane=+5VD: a +5VD plane on In4 whose pads get their own vias before routing
  (stage 1 left 14 instead of 35)
- finish.py: escape lanes kept clear of pre-route ground vias (ADC pin 2 had been fenced in by
  six); decoupling tracks protected from rip-up; plane nets handled throughout
- finish.py fixes: an empty route that looped for hours (no empty routes, a no-progress
  guard); row-at-a-time marking and A* search; KiCad's own dead ends removed

Journal, README and spec updated with the result.

Co-Authored-By: Claude Opus 5.5 <noreply@anthropic.com>
Parts:
- removed TP701: SDA, TestPoint:TestPoint_Pad_D1.0mm, symbol Connector:TestPoint
- removed TP702: SCL, TestPoint:TestPoint_Pad_D1.0mm, symbol Connector:TestPoint
- removed TP703: EXP_INT, TestPoint:TestPoint_Pad_D1.0mm, symbol Connector:TestPoint
- J714: value Holes, right top -> Holes, right middle
- J715: value Holes, right middle -> Holes, right top
Connections:
- net SW6: now also J715.1 (Pin_1); no longer J714.1 (Pin_1)
- net SW7: now also J715.2 (Pin_2); no longer J714.2 (Pin_2)
- net SW8: now also J714.1 (Pin_1); no longer J715.1 (Pin_1)
- net SW9: now also J714.2 (Pin_2); no longer J715.2 (Pin_2)
