File: hardware/analogue_board/pico_core_midi/pots_gates.kicad_sch (KiCad schematic)
At the start: 49 parts, among them J603 Gate expansion: QH', SRCLK, R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, J610 Holes, left top, J611 Holes, left bottom, J612 Holes, left top, J613 Holes, left bottom, J614 Holes, right top, J615 Holes, right middle, U601 MCP3208-CI/SL, U602 74HCT595PW

Commit message: Analogue board: the Pico board routes completely
pico_core_midi (Pico 2 / ESP32-P4, the core set with MIDI) routes with no unconnected item
and no copper fault, and every IC supply pin within 4 mm of its capacitor. Routed board in
pico_core_midi/routed_trial/, labels and wiring map, JLC files in pico_core_midi/fab/. Held:
David orders it after the Teensy board's bring-up.

What got it there:
- David's re-laid top: no chip over another on the opposite face (ADC lowered, DAC and CV
  op-amp turned and stacked, DG412s and U504 where nothing is above them, U203 moved out);
  the right-top wiring bank into the right strip's gap; no bus test points; U204 out from
  under the module
- autoroute.py --plane=+5VD: a +5VD plane on In4 whose pads get their own vias before routing
  (stage 1 left 14 instead of 35)
- finish.py: escape lanes kept clear of pre-route ground vias (ADC pin 2 had been fenced in by
  six); decoupling tracks protected from rip-up; plane nets handled throughout
- finish.py fixes: an empty route that looped for hours (no empty routes, a no-progress
  guard); row-at-a-time marking and A* search; KiCad's own dead ends removed

Journal, README and spec updated with the result.

Co-Authored-By: Claude Opus 5.5 <noreply@anthropic.com>
Parts:
- removed J615: Holes, right middle, analogue_board:WiringHoles_1x01, symbol Connector_Generic:Conn_01x01
- removed TP601: SPIB_SCK, TestPoint:TestPoint_Pad_D1.0mm, symbol Connector:TestPoint
- removed TP602: SPIB_MOSI, TestPoint:TestPoint_Pad_D1.0mm, symbol Connector:TestPoint
- removed TP603: SPIB_MISO, TestPoint:TestPoint_Pad_D1.0mm, symbol Connector:TestPoint
- removed TP604: CS_595, TestPoint:TestPoint_Pad_D1.0mm, symbol Connector:TestPoint
- removed TP605: CS_POT, TestPoint:TestPoint_Pad_D1.0mm, symbol Connector:TestPoint
- added J615, J616: Holes, right top, analogue_board:WiringHoles_1x02, symbol Connector_Generic:Conn_01x02
- J614: value Holes, right top -> Holes, right middle; footprint analogue_board:WiringHoles_1x04 -> analogue_board:WiringHoles_1x01; symbol Connector_Generic:Conn_01x04 -> Connector_Generic:Conn_01x01
Connections:
- net GOUT3: now also J616.2 (Pin_2); no longer J614.4 (Pin_4)
- net GOUT4: now also J614.1 (Pin_1)
- net POT5: now also J615.1 (Pin_1); no longer J614.1 (Pin_1)
- net POT6: now also J615.2 (Pin_2); no longer J614.2 (Pin_2)
- net POT_REF: now also J616.1 (Pin_1); no longer J614.3 (Pin_3)
